File: smb/v0.0/power.sch (KiCad schematic (older format))
At the start: 28 parts, among them P1 CONN_2, P301 CONN_2, U202 LM1117IMP-3.3, U302 MP2562DS

Commit message: Corrected production mistakes. SPI_CLK for ISP, MISO sdcard
Other:
- note added: "LM/NCP1117 and not \nMCP1826 crap from Microchip."
Changed lines of the file:
@@
-EESchema Schematic File Version 2  date jeu. 13 sept. 2012 22:24:34 CEST
+EESchema Schematic File Version 2  date 10/02/2013 13:01:35
 LIBS:power
 LIBS:device
@@
 EELAYER 25  0
 EELAYER END
-$Descr A4 11693 8268
+$Descr A4 11700 8267
 encoding utf-8
 Sheet 3 4
 Title "Short Main Board - SMB controler"
-Date "10 sep 2012"
+Date "10 feb 2013"
 Rev "0"
 Comp "XPLDUINO project"
@@
 Comment4 ""
 $EndDescr
+Text Notes 9050 600  0    60   ~ 0
+LM/NCP1117 and not \nMCP1826 crap from Microchip.
 Connection ~ 4500 2250
 Wire Wire Line
@@
 F 0 "C312" H 8325 3400 30  0000 L CNN
 F 1 "4.7uF" H 8325 3300 30  0000 L CNN
-F 2 "SM0805" H 8325 3400 30  0000 C CNN
+F 2 "SM0805" H 8325 3400 30  0001 C CNN
 	1    8300 3350
 	1    0    0    -1
@@
 F 0 "C311" H 6675 2550 30  0000 L CNN
 F 1 "1uF" H 6675 2450 30  0000 L CNN
-F 2 "SM0805" H 6675 2550 30  0000 C CNN
+F 2 "SM0805" H 6675 2550 30  0001 C CNN
 F 4 "25V" H 6900 2450 60  0000 C CNN "Volt"
 	1    6650 2500
@@
 F 0 "C310" H 6475 2550 30  0000 L CNN
 F 1 "1uF" H 6475 2450 30  0000 L CNN
-F 2 "SM0805" H 6475 2550 30  0000 C CNN
+F 2 "SM0805" H 6475 2550 30  0001 C CNN
 	1    6450 2500
 	1    0    0    -1
@@
 F 0 "C304" H 6275 2550 30  0000 L CNN
 F 1 "1uF" H 6275 2450 30  0000 L CNN
-F 2 "SM0805" H 6275 2550 30  0000 C CNN
+F 2 "SM0805" H 6275 2550 30  0001 C CNN
 	1    6250 2500
 	1    0    0    -1
@@
 F 0 "C303" H 6075 2550 30  0000 L CNN
 F 1 "1uF" H 6075 2450 30  0000 L CNN
-F 2 "SM0805" H 6075 2550 30  0000 C CNN
+F 2 "SM0805" H 6075 2550 30  0001 C CNN
 	1    6050 2500
 	1    0    0    -1
@@
 F 0 "C301" H 5875 2550 30  0000 L CNN
 F 1 "1uF" H 5875 2450 30  0000 L CNN
-F 2 "SM0805" H 5875 2550 30  0000 C CNN
+F 2 "SM0805" H 5875 2550 30  0001 C CNN
 	1    5850 2500
 	1    0    0    -1
@@
 F 0 "C308" H 9125 3400 30  0000 L CNN
 F 1 "4.7uF" H 9125 3300 30  0000 L CNN
-F 2 "SM0805" H 9125 3400 30  0000 C CNN
+F 2 "SM0805" H 9125 3400 30  0001 C CNN
 F 4 "16V" H 9400 3300 60  0000 C CNN "Volt"
 	1    9100 3350
@@
 F 0 "C307" H 8925 3400 30  0000 L CNN
 F 1 "4.7uF" H 8925 3300 30  0000 L CNN
-F 2 "SM0805" H 8925 3400 30  0000 C CNN
+F 2 "SM0805" H 8925 3400 30  0001 C CNN
 	1    8900 3350
 	1    0    0    -1
@@
 F 0 "C306" H 8725 3400 30  0000 L CNN
 F 1 "4.7uF" H 8725 3300 30  0000 L CNN
-F 2 "SM0805" H 8725 3400 30  0000 C CNN
+F 2 "SM0805" H 8725 3400 30  0001 C CNN
 	1    8700 3350
 	1    0    0    -1
@@
 F 0 "C305" H 8525 3400 30  0000 L CNN
 F 1 "4.7uF" H 8525 3300 30  0000 L CNN
-F 2 "SM0805" H 8525 3400 30  0000 C CNN
+F 2 "SM0805" H 8525 3400 30  0001 C CNN
 	1    8500 3350
 	1    0    0    -1
@@
 F 0 "R301" V 5080 3150 50  0000 C CNN
 F 1 "17.4k" V 5000 3150 50  0000 C CNN
-F 2 "SM0603" V 5100 3150 50  0000 C CNN
+F 2 "SM0603" V 5100 3150 50  0001 C CNN
 	1    5000 3150
 	1    0    0    -1
@@
 F 0 "R302" V 5330 2650 50  0000 C CNN
 F 1 "100k" V 5250 2650 50  0000 C CNN
-F 2 "SM0603" V 5350 2650 50  0000 C CNN
+F 2 "SM0603" V 5350 2650 50  0001 C CNN
 	1    5250 2650
 	1    0    0    -1
@@
 F 0 "R304" V 6030 4350 50  0000 C CNN
 F 1 "158k" V 5950 4350 50  0000 C CNN
-F 2 "SM0603" V 6050 4350 50  0000 C CNN
+F 2 "SM0603" V 6050 4350 50  0001 C CNN
 	1    5950 4350
 	1    0    0    -1
@@
 F 0 "R305" V 6430 3600 50  0000 C CNN
 F 1 "40.2k" V 6350 3600 50  0000 C CNN
-F 2 "SM0603" V 6450 3600 50  0000 C CNN
+F 2 "SM0603" V 6450 3600 50  0001 C CNN
 	1    6350 3600
 	1    0    0    -1
@@
 F 0 "R303" V 5480 3550 50  0000 C CNN
 F 1 "200k" V 5400 3550 50  0000 C CNN
-F 2 "SM0603" V 5500 3550 50  0000 C CNN
+F 2 "SM0603" V 5500 3550 50  0001 C CNN
 	1    5400 3550
 	1    0    0    -1
