File: in4dim4_acdc_i2c/v0.0/4DIM_4IN_ACDC_I2C.sch (KiCad schematic (older format))
At the start: 107 parts, among them IC1 ATTINY2313-P, IC2 MOC3021S, IC3 MOC3021S, IC4 MOC3021S, IC5 MOC3021S, IC6 P620, P10 CONN_2, P11 CONN_2, P12 CONN_2, P13 CONN_2, P14 CONN_2, P15 CONN_2, P4 CONN_5, P5 CONN_5, P6 CONN_5, P7 CONN_2, P8 CONN_2, P9 CONN_2, U1 TRIAC, U2 TRIAC, U3 TRIAC, U4 TRIAC

Commit message: Dimmer AC: Remove all the pull-up resistors (we will use the internal pull up resistors of the ATTiny)
Parts:
- removed R10, R11, R12, R9: 4.7KR, symbol R
- removed R16: 10KR, symbol R
- removed R30: 3KR, symbol R
- KUA0, KUA1, KUA2, KUA3: symbol CONN_3 -> CONN_2
