File: smb/v0.1/ethernet.sch (KiCad schematic (older format))
At the start: 22 parts, among them J401 HR911105_RJ45, U201 ENC28J60, U301 74HC08, X201 25MHz

Commit message: modif schema
Connections:
- no-connect marks 0 -> 1
Changed lines of the file:
@@
-EESchema Schematic File Version 2  date lun. 13 mai 2013 21:16:35 CEST
+EESchema Schematic File Version 2  date mar. 14 mai 2013 12:19:51 CEST
 LIBS:power
 LIBS:device
@@
 LIBS:ALPS_SWITCHS
 LIBS:SMB-cache
-EELAYER 27 0
+EELAYER 24 0
 EELAYER END
 $Descr A4 11693 8268
@@
 Sheet 4 4
 Title "Short Main Board - SMB controler"
-Date "13 may 2013"
+Date "14 may 2013"
 Rev "0"
 Comp "XPLDUINO project"
@@
 F 0 "J401" H 10200 3850 60  0000 C CNN
 F 1 "HR911105_RJ45" V 10600 3350 60  0000 C CNN
+F 2 "" H 10050 3200 60  0001 C CNN
+F 3 "" H 10050 3200 60  0001 C CNN
 	1    10050 3200
 	1    0    0    -1
@@
 F 0 "R402" V 8530 4550 50  0000 C CNN
 F 1 "270R" V 8450 4550 50  0000 C CNN
+F 2 "" H 8450 4550 60  0001 C CNN
+F 3 "" H 8450 4550 60  0001 C CNN
 	1    8450 4550
 	0    -1   -1   0
@@
 F 0 "R401" V 8530 4350 50  0000 C CNN
 F 1 "270R" V 8450 4350 50  0000 C CNN
+F 2 "" H 8450 4350 60  0001 C CNN
+F 3 "" H 8450 4350 60  0001 C CNN
 	1    8450 4350
 	0    -1   -1   0
 $EndComp
 $Comp
-L +5V #PWR066
+L +5V #PWR078
 U 1 1 4FDE1BE4
 P 7500 4300
-F 0 "#PWR066" H 7500 4390 20  0001 C CNN
+F 0 "#PWR078" H 7500 4390 20  0001 C CNN
 F 1 "+5V" H 7500 4390 30  0000 C CNN
+F 2 "" H 7500 4300 60  0001 C CNN
+F 3 "" H 7500 4300 60  0001 C CNN
 	1    7500 4300
 	1    0    0    -1
 $EndComp
 $Comp
-L GND #PWR067
+L GND #PWR079
 U 1 1 4FDE1B8D
 P 7500 5100
-F 0 "#PWR067" H 7500 5100 30  0001 C CNN
+F 0 "#PWR079" H 7500 5100 30  0001 C CNN
 F 1 "GND" H 7500 5030 30  0001 C CNN
+F 2 "" H 7500 5100 60  0001 C CNN
+F 3 "" H 7500 5100 60  0001 C CNN
 	1    7500 5100
 	1    0    0    -1
 $EndComp
 $Comp
-L GND #PWR068
+L GND #PWR080
 U 1 1 4FDE1B70
 P 3000 2750
-F 0 "#PWR068" H 3000 2750 30  0001 C CNN
+F 0 "#PWR080" H 3000 2750 30  0001 C CNN
 F 1 "GND" H 3000 2680 30  0001 C CNN
+F 2 "" H 3000 2750 60  0001 C CNN
+F 3 "" H 3000 2750 60  0001 C CNN
 	1    3000 2750
 	1    0    0    -1
 $EndComp
 $Comp
-L +5V #PWR069
+L +5V #PWR081
 U 1 1 4FDE1B61
 P 2850 3400
-F 0 "#PWR069" H 2850 3490 20  0001 C CNN
+F 0 "#PWR081" H 2850 3490 20  0001 C CNN
 F 1 "+5V" H 2850 3490 30  0000 C CNN
+F 2 "" H 2850 3400 60  0001 C CNN
+F 3 "" H 2850 3400 60  0001 C CNN
 	1    2850 3400
 	-1   0    0    1
@@
 F 0 "U301" H 7700 4850 60  0000 C CNN
 F 1 "74HC08" H 7700 4750 60  0000 C CNN
+F 2 "" H 7700 4800 60  0001 C CNN
+F 3 "" H 7700 4800 60  0001 C CNN
 	2    7700 4800
 	1    0    0    -1
@@
 F 0 "U301" H 2650 3050 60  0000 C CNN
 F 1 "74HC08" H 2650 2950 60  0000 C CNN
+F 2 "" H 2650 3000 60  0001 C CNN
+F 3 "" H 2650 3000 60  0001 C CNN
 	1    2650 3000
 	-1   0    0    1
@@
 F 1 "50" V 7450 2500 50  0000 C CNN
 F 2 "SM0603" V 7550 2500 50  0001 C CNN
+F 3 "" H 7450 2500 60  0001 C CNN
 	1    7450 2500
 	1    0    0    -1
@@
 F 1 "50" V 7250 2500 50  0000 C CNN
 F 2 "SM0603" V 7350 2500 50  0001 C CNN
+F 3 "" H 7250 2500 60  0001 C CNN
 	1    7250 2500
 	1    0    0    -1
@@
 F 0 "L201" V 8500 1850 40  0000 C CNN
 F 1 "4.7uH" V 8650 1850 40  0000 C CNN
+F 2 "" H 8550 1850 60  0001 C CNN
+F 3 "" H 8550 1850 60  0001 C CNN
 	1    8550 1850
 	1    0    0    -1
 $EndComp
 $Comp
-L +3.3V #PWR070
+L +3.3V #PWR082
 U 1 1 4FA00F89
 P 8550 1500
-F 0 "#PWR070" H 8550 1460 30  0001 C CNN
+F 0 "#PWR082" H 8550 1460 30  0001 C CNN
 F 1 "+3.3V" H 8550 1610 30  0000 C CNN
+F 2 "" H 8550 1500 60  0001 C CNN
+F 3 "" H 8550 1500 60  0001 C CNN
 	1    8550 1500
 	1    0    0    -1
 $EndComp
 $Comp
-L GND #PWR071
+L GND #PWR083
 U 1 1 4FA00F53
 P 8550 3700
-F 0 "#PWR071" H 8550 3700 30  0001 C CNN
+F 0 "#PWR083" H 8550 3700 30  0001 C CNN
 F 1 "GND" H 8550 3630 30  0001 C CNN
+F 2 "" H 8550 3700 60  0001 C CNN
+F 3 "" H 8550 3700 60  0001 C CNN
 	1    8550 3700
 	1    0    0    -1
@@
 F 1 "100nF" H 8600 3300 50  0000 L CNN
 F 2 "SM0603" H 8600 3400 50  0000 C CNN
+F 3 "" H 8550 3400 60  0001 C CNN
 	1    8550 3400
 	1    0    0    -1
 $EndComp
 $Comp
-L GND #PWR072
+L GND #PWR084
 U 1 1 4FA00C7B
 P 9450 3900
-F 0 "#PWR072" H 9450 3900 30  0001 C CNN
+F 0 "#PWR084" H 9450 3900 30  0001 C CNN
 F 1 "GND" H 9450 3830 30  0001 C CNN
+F 2 "" H 9450 3900 60  0001 C CNN
+F 3 "" H 9450 3900 60  0001 C CNN
 	1    9450 3900
 	1    0    0    -1
 $EndComp
 $Comp
-L GND #PWR073
+L GND #PWR085
 U 1 1 4FA00C63
 P 10650 4000
-F 0 "#PWR073" H 10650 4000 30  0001 C CNN
+F 0 "#PWR085" H 10650 4000 30  0001 C CNN
 F 1 "GND" H 10650 3930 30  0001 C CNN
+F 2 "" H 10650 4000 60  0001 C CNN
+F 3 "" H 10650 4000 60  0001 C CNN
 	1    10650 4000
 	1    0    0    -1
 $EndComp
 $Comp
-L GND #PWR074
+L GND #PWR086
 U 1 1 4F9FF676
 P 7800 4250
-F 0 "#PWR074" H 7800 4250 30  0001 C CNN
+F 0 "#PWR086" H 7800 4250 30  0001 C CNN
 F 1 "GND" H 7800 4180 30  0001 C CNN
+F 2 "" H 7800 4250 60  0001 C CNN
+F 3 "" H 7800 4250 60  0001 C CNN
 	1    7800 4250
 	1    0    0    -1
@@
 F 1 "100nF" H 7850 3850 50  0000 L CNN
 F 2 "SM0603" H 7850 3950 50  0000 C CNN
+F 3 "" H 7800 3950 60  0001 C CNN
 	1    7800 3950
 	1    0    0    -1
@@
 F 1 "50" V 7900 3300 50  0000 C CNN
 F 2 "SM0603" V 8000 3300 50  0001 C CNN
+F 3 "" H 7900 3300 60  0001 C CNN
 	1    7900 3300
 	1    0    0    -1
@@
 F 1 "50" V 7700 3400 50  0000 C CNN
 F 2 "SM0603" V 7800 3400 50  0001 C CNN
+F 3 "" H 7700 3400 60  0001 C CNN
 	1    7700 3400
 	1    0    0    -1
@@
 SPI_CLK
 $Comp
-L GND #PWR075
+L GND #PWR087
 U 1 1 4F9FEE21
 P 3400 4200
-F 0 "#PWR075" H 3400 4200 30  0001 C CNN
+F 0 "#PWR087" H 3400 4200 30  0001 C CNN
 F 1 "GND" H 3400 4130 30  0001 C CNN
+F 2 "" H 3400 4200 60  0001 C CNN
+F 3 "" H 3400 4200 60  0001 C CNN
 	1    3400 4200
 	1    0    0    -1
 $EndComp
 $Comp
-L GND #PWR076
+L GND #PWR088
 U 1 1 4F9FEE1E
 P 4000 4400
-F 0 "#PWR076" H 4000 4400 30  0001 C CNN
+F 0 "#PWR088" H 4000 4400 30  0001 C CNN
 F 1 "GND" H 4000 4330 30  0001 C CNN
+F 2 "" H 4000 4400 60  0001 C CNN
+F 3 "" H 4000 4400 60  0001 C CNN
 	1    4000 4400
 	1    0    0    -1
@@
 F 1 "2k7" H 4150 4200 50  0000 C CNN
 F 2 "SM0603" H 4150 4300 50  0000 C CNN
+F 3 "" H 4000 4050 60  0001 C CNN
 	1    4000 4050
 	1    0    0    -1
@@
 F 1 "10uF" H 3450 3700 50  0000 L CNN
 F 2 "SM0805" H 3450 3800 50  0000 C CNN
+F 3 "" H 3400 3800 60  0001 C CNN
 	1    3400 3800
 	1    0    0    -1
 $EndComp
 $Comp
-L GND #PWR077
+L GND #PWR089
 U 1 1 4F9FC462
 P 5050 2150
-F 0 "#PWR077" H 5050 2150 30  0001 C CNN
+F 0 "#PWR089" H 5050 2150 30  0001 C CNN
 F 1 "GND" H 5050 2080 30  0001 C CNN
+F 2 "" H 5050 2150 60  0001 C CNN
+F 3 "" H 5050 2150 60  0001 C CNN
 	1    5050 2150
 	1    0    0    -1
 $EndComp
 $Comp
-L GND #PWR078
+L GND #PWR090
 U 1 1 4F9FC45C
 P 6750 2100
-F 0 "#PWR078" H 6750 2100 30  0001 C CNN
+F 0 "#PWR090" H 6750 2100 30  0001 C CNN
 F 1 "GND" H 6750 2030 30  0001 C CNN
+F 2 "" H 6750 2100 60  0001 C CNN
+F 3 "" H 6750 2100 60  0001 C CNN
 	1    6750 2100
 	1    0    0    -1
@@
 F 1 "0.1uF" V 5350 2100 50  0000 L CNN
 F 2 "SM0603" H 5350 1750 60  0000 C CNN
+F 3 "" H 5350 1750 60  0001 C CNN
 	1    5350 1750
 	0    -1   -1   0
@@
 F 1 "0.1uF" V 5350 2350 50  0000 L CNN
 F 2 "SM0603" H 5350 2000 60  0000 C CNN
+F 3 "" H 5350 2000 60  0001 C CNN
 	1    5350 2000
 	0    -1   -1   0
@@
 F 1 "0.1uF" V 6450 1450 50  0000 L CNN
 F 2 "SM0603" H 6450 2000 60  0000 C CNN
+F 3 "" H 6450 2000 60  0001 C CNN
 	1    6450 2000
 	0    -1   -1   0
@@
 F 1 "0.1uF" V 6450 1200 50  0000 L CNN
 F 2 "SM0603" H 6450 1750 60  0000 C CNN
+F 3 "" H 6450 1750 60  0001 C CNN
 	1    6450 1750
 	0    -1   -1   0
@@
 F 1 "0.1uF" V 6450 950 50  0000 L CNN
 F 2 "SM0603" H 6450 1500 60  0000 C CNN
+F 3 "" H 6450 1500 60  0001 C CNN
 	1    6450 1500
 	0    -1   -1   0
 $EndComp
 $Comp
-L +3.3V #PWR079
+L +3.3V #PWR091
 U 1 1 4F9FC2EE
 P 5900 1450
-F 0 "#PWR079" H 5900 1410 30  0001 C CNN
+F 0 "#PWR091" H 5900 1410 30  0001 C CNN
 F 1 "+3.3V" H 5900 1560 30  0000 C CNN
+F 2 "" H 5900 1450 60  0001 C CNN
+F 3 "" H 5900 1450 60  0001 C CNN
 	1    5900 1450
 	1    0    0    -1
 $EndComp
 $Comp
-L GND #PWR080
+L GND #PWR092
 U 1 1 4F9D7261
 P 4350 5050
-F 0 "#PWR080" H 4350 5050 30  0001 C CNN
+F 0 "#PWR092" H 4350 5050 30  0001 C CNN
 F 1 "GND" H 4350 4980 30  0001 C CNN
+F 2 "" H 4350 5050 60  0001 C CNN
+F 3 "" H 4350 5050 60  0001 C CNN
 	1    4350 5050
 	1    0    0    -1
 $EndComp
 $Comp
-L GND #PWR081
+L GND #PWR093
 U 1 1 4F9D725B
 P 4950 5050
-F 0 "#PWR081" H 4950 5050 30  0001 C CNN
+F 0 "#PWR093" H 4950 5050 30  0001 C CNN
 F 1 "GND" H 4950 4980 30  0001 C CNN
+F 2 "" H 4950 5050 60  0001 C CNN
+F 3 "" H 4950 5050 60  0001 C CNN
 	1    4950 5050
 	1    0    0    -1
@@
 F 1 "18pF" H 5000 4650 50  0000 L CNN
 F 2 "SM0603" H 5000 4750 50  0000 C CNN
+F 3 "" H 4950 4750 60  0001 C CNN
 	1    4950 4750
 	1    0    0    -1
@@
 F 1 "18pF" H 4400 4650 50  0000 L CNN
 F 2 "SM0603" H 4400 4750 50  0000 C CNN
+F 3 "" H 4350 4750 60  0001 C CNN
 	1    4350 4750
 	1    0    0    -1
@@
 F 0 "X201" H 4650 4550 60  0000 C CNN
 F 1 "25MHz" H 4650 4250 60  0000 C CNN
+F 2 "" H 4650 4400 60  0001 C CNN
+F 3 "" H 4650 4400 60  0001 C CNN
 	1    4650 4400
 	1    0    0    -1
 $EndComp
 $Comp
-L GND #PWR082
+L GND #PWR094
 U 1 1 4F9D6E29
 P 5850 4950
-F 0 "#PWR082" H 5850 4950 30  0001 C CNN
+F 0 "#PWR094" H 5850 4950 30  0001 C CNN
 F 1 "GND" H 5850 4880 30  0001 C CNN
+F 2 "" H 5850 4950 60  0001 C CNN
+F 3 "" H 5850 4950 60  0001 C CNN
 	1    5850 4950
 	1    0    0    -1
@@
 F 0 "U201" H 6200 4650 60  0000 L CNN
 F 1 "ENC28J60" H 6150 2400 60  0000 L CNN
+F 2 "" H 5800 3500 60  0001 C CNN
+F 3 "" H 5800 3500 60  0001 C CNN
 	1    5800 3500
 	1    0    0    -1
 $EndComp
+NoConn ~ 9500 2800
 $EndSCHEMATC
