File: smb/v0.1/power.sch (KiCad schematic (older format))
At the start: 28 parts, among them P1 CONN_2, P301 CONN_2, U202 LM1117IMP-3.3, U302 MP2562DS

Commit message: routage complet ajout rs485 attention, tous les packages sont ? v?rifier
Connections:
- net labels added: pre_5V
