File: smb/v0.1/power.sch (KiCad schematic (older format))
At the start: 28 parts, among them P1 CONN_2, P301 CONN_2, U202 LM1117IMP-3.3, U302 MP2562DS

Commit message: correction broche 8 du module RS485 + inversion tx+/tx- au niveau du connecteur + pilotage E/R independant inversion polarit? connecteur d'alim d?placement slot pour rtc simplification routage et optimisation plan de masse (affinage zone exclusion)
Connections:
- net labels added: 3.3V
