File: smb/v0.1/uSD_card.sch (KiCad schematic (older format))
At the start: 6 parts, among them J202 USD_CONN, U203 74LVC1G126GW, U204 74LVC1G126GW, U205 74LVC1G126GW, U206 74LVC1G126GW

Commit message: correction broche 8 du module RS485 + inversion tx+/tx- au niveau du connecteur + pilotage E/R independant inversion polarit? connecteur d'alim d?placement slot pour rtc simplification routage et optimisation plan de masse (affinage zone exclusion)
Parts:
- removed U203, U204, U205, U206: 74LVC1G126GW, SOT353, symbol 74LVC1G126GW
- added U301, U303: 74HC08, symbol 74HC08
Connections:
- wire segments 37 -> 28
- no-connect marks 0 -> 2
Other:
- note removed: "3.3V -> 5V"
- note removed: "5V -> 3.3V"
- note removed: "Need to tie OE to ground to \nhave a high impedance output !"
- moved on the sheet: J202
