File: 8in8out/_autosave-8in8out.kicad_pcb (KiCad board)
At the start: 2 copper layers, 122 parts, among them IC1 ATTINY2313-P, J1 RJ45, J2 RJ45, J3 CONN_6, K110 G5T-1-12VDC, K120 G5T-1-12VDC, K130 G5T-1-12VDC, K140 G5T-1-12VDC, K150 G5T-1-12VDC, K160 G5T-1-12VDC, K170 G5T-1-12VDC, K180 G5T-1-12VDC, P1 CONN_5, P100 CONN_2, P101 CONN_2, P102 CONN_2, P103 CONN_2, P105 CONN_2, P106 CONN_2, P107 CONN_3, P109 CONN_2, P110 CONN_2, P120 CONN_2, P130 CONN_2, P140 CONN_2, P150 CONN_2, P160 CONN_2, P170 CONN_2, P180 CONN_2, P2 CONN_5, Q110 NPN, Q120 NPN, Q130 NPN, Q140 NPN, Q150 NPN, Q160 NPN, Q170 NPN, Q180 NPN, U1 74HC595, U10 OPTO-TRANSISTOR, U2 74LS165, U20 OPTO-TRANSISTOR, U30 OPTO-TRANSISTOR, U40 OPTO-TRANSISTOR, U50 OPTO-TRANSISTOR, U60 OPTO-TRANSISTOR, U70 OPTO-TRANSISTOR, U80 OPTO-TRANSISTOR

Commit message: Draft PCB SMBV0.1
Parts:
- removed D10, D110, D120, D130, D140, D150, D160, D170, D180, D20, D30, D40, D50, D60, D70, D80: LED, LED-1206
- removed D111, D121, D131, D141, D151, D161, D171, D181: DIODE, SM1206
- removed P107: CONN_3, PIN_ARRAY_3X1
- removed P109: CONN_2, PIN_ARRAY_2X1
- removed Q110, Q120, Q130, Q140, Q150, Q160, Q170, Q180: NPN, SOT23EBC
- removed R10, R110, R111, R12, R120, R121, R130, R131, R140, R141, R150, R151, R160, R161, R170, R171, R180, R181, R20, R22, R30, R32, R40, R42, R50, R52, R60, R62, R70, R72, R80, R82: R, SM1206
- added G***: LOGO, OSHWLOGO0.3IN, F.Cu at (227.8, 89.4)
- added P3: CONN_10X2, pin_array_10x2, F.Cu at (209.9, 120.4)
- added P4: CONN_2, PIN_ARRAY_2X1, F.Cu at (259.3, 133.9)
- added R5: 10KR, SM1206, F.Cu at (270.8, 121.9)
- added R6: 10KR, SM1206, F.Cu at (268.2, 121.9)
- added logo_xplduino: VAL**, logo_xplduino, F.Cu at (192.0, 112.4)
- added logo_xplduino: VAL**, logo_xplduino, B.Cu at (231.4, 92.7)
- IC1: value ATTINY2313-P -> ATTINY48-A; footprint SO20L -> TQFP32
- P105: footprint PIN_ARRAY_2X1 -> MOL_CONN_2_MINI
- R1, R11, R21, R3, R31, R41, R51, R61, R71, R81: value R -> 2KR
- R2: value R -> 4.7KR
- R4: value R -> 10KR
- U1: value 74HC595 -> 7805; footprint SO16E -> TO220_7805_VERT; moved to F.Cu
- U2: value 74LS165 -> ULN2803; footprint SO16E -> SOIC18; moved to F.Cu
- moved R1 216.7 mm to (278.4, 121.9), turned to 90 degrees
- moved C2 214.2 mm to (275.8, 121.9), turned to 90 degrees
- moved D1 214.1 mm to (276.4, 115.6), turned to 90 degrees
- moved P106 213.5 mm to (276.1, 110.6)
- moved D2 211.8 mm to (274.1, 115.6), turned to 90 degrees
- moved C1 211.7 mm to (273.3, 121.9), turned to 90 degrees
- moved R2 206.3 mm to (268.5, 115.6), turned to 270 degrees
- moved R4 204.1 mm to (265.7, 121.9), turned to 90 degrees
- moved R3 201.6 mm to (263.1, 121.9), turned to 90 degrees
- moved D3 198.9 mm to (260.5, 121.9), turned to 90 degrees
- moved P100 193.0 mm to (253.9, 126.5), turned to 90 degrees
- moved P101 190.5 mm to (251.3, 126.5), turned to 90 degrees
- moved P102 187.9 mm to (248.8, 126.5), turned to 90 degrees
- moved P105 185.8 mm to (241.6, 149.7)
- moved P103 185.4 mm to (246.3, 126.5), turned to 90 degrees
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Connections:
- C1 pad 2: DGND -> GND
- C2 pad 2: DGND -> GND
- D1 pad 2: DGND -> GND
- D2 pad 2: DGND -> GND
- D3 pad 1: N-0000035 -> LED
- IC1 pad 1: N-0000031 -> A0
- IC1 pad 10: DGND -> OUT7
- IC1 pad 11: /INT -> OUT3
- IC1 pad 12: DATA_IN -> OUT2
- IC1 pad 13: A0 -> OUT1
- IC1 pad 14: A1 -> OUT0
- IC1 pad 15: A2 -> MOSI
- IC1 pad 16: A3 -> MISO
- IC1 pad 17: MOSI(SDA) -> SCK
- IC1 pad 18: MISO -> +5V
- IC1 pad 19: SCK(SCL) -> CMD7
- IC1 pad 2: RX -> A1
- IC1 pad 20: +5V -> CMD6
- IC1 pad 3: TX -> A2
- IC1 pad 4: LATCH_IN -> +5V
- IC1 pad 5: N-0000035 -> GND
- IC1 pad 6: CLK_IN -> A3
- IC1 pad 7: (no net) -> OUT4
- IC1 pad 8: (no net) -> OUT5
- IC1 pad 9: (no net) -> OUT6
- ISP0 pad 1: (no net) -> RESET
- ISP0 pad 2: DGND -> GND
- ISP0 pad 3: SCK(SCL) -> SCK
- ISP0 pad 4: MOSI(SDA) -> MOSI
- J1 pad 1: MOSI(SDA) -> SDA
- J1 pad 2: DGND -> GND
- J1 pad 3: SCK(SCL) -> SCL
- J1 pad 4: DGND -> GND
- J1 pad 6: DGND -> GND
- J1 pad 7: +5V -> 5V_EXT
- J1 pad 8: +5V -> 5V_EXT
- J2 pad 1: MOSI(SDA) -> SDA
- J2 pad 2: DGND -> GND
- J2 pad 3: SCK(SCL) -> SCL
- J2 pad 4: DGND -> GND
- J2 pad 6: DGND -> GND
- J2 pad 7: +5V -> 5V_EXT
- J2 pad 8: +5V -> 5V_EXT
- J3 pad 1: +5V -> 5V_EXT
- J3 pad 2: DGND -> GND
- J3 pad 3: SCK(SCL) -> SCL
- J3 pad 4: MOSI(SDA) -> SDA
- K110 pad 2: N-0000032 -> R0
- K120 pad 2: N-000004 -> R1
- K130 pad 2: N-000001 -> R2
- K140 pad 2: N-000007 -> R3
- K150 pad 2: N-0000024 -> R4
- K160 pad 2: N-0000028 -> R5
- K170 pad 2: N-0000014 -> R6
- K180 pad 2: N-0000021 -> R7
- P1 pad 5: GND -> COM0
- P100 pad 1: DGND -> GND
- P101 pad 1: DGND -> GND
- P102 pad 1: DGND -> GND
- P103 pad 1: DGND -> GND
- P105 pad 2: DGND -> GND
- P106 pad 2: DGND -> GND
- P2 pad 5: GND -> COM1
- R11 pad 2: GND -> COM0
- R21 pad 2: GND -> COM0
- R3 pad 2: DGND -> GND
- R31 pad 2: GND -> COM0
- R4 pad 2: N-0000031 -> RESET
- R41 pad 2: GND -> COM0
- R51 pad 2: GND -> COM1
- R61 pad 2: GND -> COM1
- R71 pad 2: GND -> COM1
- R81 pad 2: GND -> COM1
- U10 pad 4: DGND -> GND
- U2 pad 1: LATCH_IN -> OUT0
- U2 pad 10: DATA_IN -> +12V
- U2 pad 11: CMD0 -> R7
- U2 pad 12: CMD1 -> R6
- U2 pad 13: CMD2 -> R5
- U2 pad 14: CMD3 -> R4
- U2 pad 15: CLK_IN -> R3
- U2 pad 16: +5V -> R2
- U2 pad 2: CLK_IN -> OUT1
- U2 pad 3: CMD4 -> OUT2
- U2 pad 4: CMD5 -> OUT3
- U2 pad 5: CMD6 -> OUT4
- U2 pad 6: CMD7 -> OUT5
- U2 pad 7: (no net) -> OUT6
- U2 pad 8: GND -> OUT7
- U2 pad 9: (no net) -> GND
- U20 pad 4: DGND -> GND
- U30 pad 4: DGND -> GND
- U40 pad 4: DGND -> GND
- U50 pad 4: DGND -> GND
- U60 pad 4: DGND -> GND
- U70 pad 4: DGND -> GND
- U80 pad 4: DGND -> GND
Routing:
- net +12V: track 0.00 -> 174.8 mm, vias 0 -> 1
- net +5V: track 0.00 -> 101.7 mm, vias 0 -> 1
- net COM0: track 0.00 -> 75.7 mm, vias 0 -> 2
- net SCL: track 0.00 -> 72.1 mm, vias 0 -> 1
- net RESET: track 0.00 -> 66.0 mm, vias 0 -> 2
- net SDA: track 0.00 -> 64.9 mm, vias 0 -> 2
- net /INT: track 0.00 -> 61.2 mm
- net LED: track 0.00 -> 59.5 mm, vias 0 -> 3
- net OUT4: track 0.00 -> 58.7 mm, vias 0 -> 1
- net OUT0: track 0.00 -> 57.6 mm, vias 0 -> 1
- net CMD1: track 0.00 -> 57.3 mm, vias 0 -> 1
- net OUT1: track 0.00 -> 56.2 mm, vias 0 -> 1
- net CMD7: track 0.00 -> 55.3 mm, vias 0 -> 1
- net OUT2: track 0.00 -> 54.7 mm, vias 0 -> 1
- net CMD6: track 0.00 -> 54.3 mm, vias 0 -> 1
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- added copper zone on B.Cu, net GND
- added copper zone on F.Cu, net GND
Other:
- net class +230 1mm: clearance 0.254 -> 1.50114
- net class +230V: clearance 0.254 -> 0.508; trace_width 0.7493 -> 2.54
- net class GND added: clearance 0.254, trace_width 0.50038, via_dia 0.889, via_drill 0.635
- board text added: "0 1 2 3"
- board text added: "1"
- board text added: "12V"
- board text added: "12V - GND"
- board text added: "12V-GND"
- board text added: "2"
- board text added: "3"
- board text added: "3 2 1 0 ID 0 0 0 0 0 0 0 0 1 1 0 1 1 0 2 0 1 1 1 3 0 0 0 0 4 0 0 0 1 5 0 1 1 0 6 0 1 1 1 7 1 0 0 0 8 1 0 0 1 9 1 1 1 0 10 1 1 1 1 11 1 0 0 0 12 1 0 0 1 13 1 1 1 0 14 1 1 1 1 15"
- board text added: "4"
- board text added: "5"
- board text added: "5V"
- board text added: "5V ext"
- board text added: "6"
- board text added: "7"
- board text added: "@I2C"
- board text added: "@I2C ID TABLE"
- board text added: "COM0"
- board text added: "COM1"
- board text added: "FRONT PANEL"
- board text added: "I2C PORT"
- board text added: "IN 0"
- board text added: "IN8R8 v0.0 I2C BOARD"
- board text added: "ISP"
- board text added: "OUT 0"
- board text added: "OUT 1"
- board text added: "OUT 2"
- board text added: "OUT 3"
- board text added: "OUT 4"
- board text added: "OUT 5"
- board text added: "OUT 6"
- board text added: "OUT 7"
- board text added: "STATUS"
- board text added: "home automation"
