File: in4dim4mosfet/v0/4in4dim.sch (KiCad schematic (older format))
At the start: 90 parts, among them IC1 ATTINY48-A, IC2 MAX485, J1 RJ45, J2 RJ45, J3 CONN_6, K1 CONN_3, P1 CONN_5, P100 CONN_2, P101 CONN_2, P102 CONN_2, P103 CONN_2, P105 CONN_2, P106 CONN_2, P110 CONN_2, P120 CONN_2, P130 CONN_2, P140 CONN_2, P2 CONN_2, P3 CONN_6X2, Q1 SPP20N60C3, Q2 SPP20N60C3, Q3 SPP20N60C3, Q4 SPP20N60C3, U1 7805, U2 LTV847, U3 LTV847

Commit message: update
Parts:
- added RP1, RP2, RP3, RP4, RP5, RP6, RP7, RP8: 0R, symbol R
Connections:
- net CMD0: now also P3.7 (P7); no longer P3.1 (P1)
- net CMD1: now also IC1.24 ((PCINT9/ADC1)PC1), P3.5 (P5); no longer IC1.26 ((PCINT11/ADC3)PC3), P3.3 (P3)
- net CMD2: now also P3.3 (P3); no longer P3.5 (P5)
- net CMD3: now also IC1.26 ((PCINT11/ADC3)PC3), P3.1 (P1); no longer IC1.24 ((PCINT9/ADC1)PC1), P3.7 (P7)
- net OUT0_A: now also RP7.2; no longer U3.16 (C)
- net OUT0_B: now also RP8.2; no longer U3.15 (E)
- net OUT1_A: now also RP5.2; no longer U3.14 (C)
- net OUT1_B: now also RP6.2; no longer U3.13 (E)
- net OUT2_A: now also RP3.2; no longer U3.12 (C)
- net OUT2_B: now also RP4.2; no longer U3.11 (E)
- net OUT3_A: now also RP1.2; no longer U3.10 (C)
- net OUT3_B: now also RP2.2; no longer U3.9 (E)
- net 130S: now reaches C131.2, C132.2, C133.2, D131.1 (-), D133.2 (K), Q3.3 (S), R133.1
- net 130D: now reaches D131.3 (+), Q3.1 (D)
- net 140S: now reaches C141.2, C142.2, C143.2, D141.1 (-), D143.2 (K), Q4.3 (S), R143.1
- net 140D: now reaches D141.3 (+), Q4.1 (D)
- new net: RP7.1, U3.10 (C)
- new net: RP6.1, U3.11 (E)
- new net: RP5.1, U3.12 (C)
- new net: RP4.1, U3.13 (E)
- new net: RP3.1, U3.14 (C)
- new net: RP2.1, U3.15 (E)
- new net: RP1.1, U3.16 (C)
- new net: RP8.1, U3.9 (E)
Other:
- moved on the sheet: R16, R17, R18, R19, U3
